File: Kicad/NE555_OC.kicad_sch (KiCad schematic)
At the start: 15 parts, among them J1 Conn_01x02_Male, J2 Conn_01x02_Male, Q1 MMBT3904, U1 NE555D, U2 AP1117-5

Commit message: Add files via upload
Parts:
- removed U2: AP1117-5, Package_TO_SOT_SMD:SOT-223-3_TabPin2, symbol Regulator_Linear:AP1117-15
- added D4: 5V6, Diode_SMD:D_MiniMELF, symbol Device:D_Zener
- added Q2: BCX56, Package_TO_SOT_SMD:SOT-89-3, symbol Transistor_BJT:BCX56
- added R4: 8k2, Resistor_SMD:R_1206_3216Metric, symbol Device:R
Connections:
- net +24V: now also Q2.2 (C), R4.1; no longer C1.1
- net +5V: now also Q2.3 (E)
- net GND: now also D4.2 (A)
- new net: C1.1, D4.1 (K), Q2.1 (B), R4.2
Other:
- moved on the sheet: C3, C4, J1
